File: Блок питания усилителя/Блок питания усилителя.kicad_pcb (KiCad board)
At the start: 2 copper layers, 20 parts, among them J1 Screw_Terminal_01x03, J2 Screw_Terminal_01x03, U2 LM7912_TO220, U3 LM7812_TO220

Commit message: Более менее рабчая версия платы
Parts:
- removed the REF** at (159.0, 84.0)
- added REF**: Heatsink, Heatsink:Heatsink_TO220_22x25x15mm_P_18mm, F.Cu at (129.0, 82.0)
- added REF**: Heatsink, Heatsink:Heatsink_TO220_22x25x15mm_P_18mm, F.Cu at (129.0, 108.0)
- C3, C4: footprint Capacitor_THT:CP_Radial_D10.0mm_P2.50mm -> Capacitor_THT:CP_Radial_D16.0mm_P7.50mm
- C5, C6: footprint Capacitor_THT:CP_Radial_D6.3mm_P2.50mm -> Capacitor_THT:CP_Radial_D8.0mm_P3.50mm
- D1: footprint Diode_THT:Diode_Bridge_32.0x5.6x17.0mm_P10.0mm_P7.5mm -> Diode_THT:Diode_Bridge_Vishay_KBL
- F1: footprint Fuse:Fuseholder_Clip-5x20mm_Littelfuse_111_Lateral_P18.80x5.00mm_D1.17mm_Horizontal -> Fuse:Fuseholder_Clip-5x20mm_Littelfuse_445-030_Inline_P20.50x5.20mm_D1.30mm_Horizontal
- F2: footprint Fuse:Fuseholder_Clip-5x20mm_Littelfuse_111_Lateral_P18.80x5.00mm_D1.17mm_Horizontal -> Fuse:Fuseholder_Clip-5x20mm_Littelfuse_520_Inline_P20.50x5.80mm_D1.30mm_Horizontal
- moved D2 76.0 mm to (97.4, 74.5), turned to 0 degrees
- moved C2 73.1 mm to (81.0, 107.5)
- moved C1 65.0 mm to (91.0, 81.0), turned to 180 degrees
- moved D3 55.5 mm to (115.1, 100.0), turned to 180 degrees
- moved D5 50.4 mm to (140.2, 84.0), turned to 0 degrees
- moved R1 48.4 mm to (138.2, 77.5), turned to 0 degrees
- moved D4 47.5 mm to (140.5, 109.5), turned to -90 degrees
- moved D1 38.1 mm to (97.1, 86.9)
- moved J1 38.0 mm to (83.5, 99.5)
- moved C4 37.8 mm to (109.0, 115.5), turned to 90 degrees
- moved F2 37.2 mm to (149.0, 105.2), turned to 90 degrees
- moved C3 35.2 mm to (111.0, 90.0), turned to 90 degrees
- moved J2 35.0 mm to (164.0, 100.0)
- moved R2 32.9 mm to (140.5, 104.8), turned to 90 degrees
- moved U2 28.5 mm to (133.0, 110.5), turned to 90 degrees
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Connections:
- C1 pad 2: Net-(J1-Pin_2) -> Net-(D4-A)
- C2 pad 1: Net-(J1-Pin_2) -> Net-(D4-A)
- C3 pad 2: Net-(J1-Pin_2) -> Net-(D4-A)
- C4 pad 1: Net-(J1-Pin_2) -> Net-(D4-A)
- C5 pad 2: Net-(J1-Pin_2) -> Net-(D4-A)
- C6 pad 1: Net-(J1-Pin_2) -> Net-(D4-A)
- D4 pad 1: Net-(D3-K) -> Net-(D4-K)
- D5 pad 1: Net-(D2-A) -> Net-(D4-A)
- J1 pad 2: Net-(J1-Pin_2) -> Net-(D4-A)
- J2 pad 2: Net-(J1-Pin_2) -> Net-(D4-A)
- R1 pad 1: Net-(D5-A) -> Net-(D2-A)
- R1 pad 2: Net-(J1-Pin_2) -> Net-(D5-A)
- R2 pad 1: Net-(J1-Pin_2) -> Net-(D4-K)
- R2 pad 2: Net-(D4-A) -> Net-(D3-K)
- U2 pad 1: Net-(J1-Pin_2) -> Net-(D4-A)
- U3 pad 2: Net-(J1-Pin_2) -> Net-(D4-A)
Routing:
- net Net-(D4-A): track 5.27 -> 237.8 mm
- net Net-(J1-Pin_2): track 108.9 -> 0.00 mm
- net Net-(D2-A): track 42.4 -> 68.1 mm
- net Net-(J2-Pin_3): track 14.1 -> 31.5 mm
- net Net-(D1--): track 40.8 -> 51.5 mm
- net Net-(J1-Pin_3): track 24.0 -> 14.6 mm
- net Net-(D4-K): track 0.00 -> 4.69 mm
- net Net-(D3-K): track 53.0 -> 57.7 mm
- net Net-(D5-A): track 4.86 -> 8.19 mm
- net Net-(J2-Pin_1): track 13.8 -> 11.9 mm
- net Net-(J1-Pin_1): track 16.5 -> 14.6 mm
- net Net-(D1-+): track 57.4 -> 56.4 mm
- added copper zone on B.Cu, net Net-(D4-A)
Other:
- board outline added: 94.5 x 52 mm
