File: Блок питания усилителя/Блок питания усилителя.kicad_sch (KiCad schematic)
At the start: 19 parts, among them J1 Screw_Terminal_01x03, J2 Screw_Terminal_01x03, U2 LM7912_TO220, U3 LM7812_TO220

Commit message: Более менее рабчая версия платы
Parts:
- C3, C4: footprint Capacitor_THT:CP_Radial_D10.0mm_P2.50mm -> Capacitor_THT:CP_Radial_D16.0mm_P7.50mm
- C5, C6: footprint Capacitor_THT:CP_Radial_D6.3mm_P2.50mm -> Capacitor_THT:CP_Radial_D8.0mm_P3.50mm
- D1: footprint Diode_THT:Diode_Bridge_32.0x5.6x17.0mm_P10.0mm_P7.5mm -> Diode_THT:Diode_Bridge_Vishay_KBL
- F1: footprint Fuse:Fuseholder_Clip-5x20mm_Littelfuse_111_Lateral_P18.80x5.00mm_D1.17mm_Horizontal -> Fuse:Fuseholder_Clip-5x20mm_Littelfuse_445-030_Inline_P20.50x5.20mm_D1.30mm_Horizontal
- F2: footprint Fuse:Fuseholder_Clip-5x20mm_Littelfuse_111_Lateral_P18.80x5.00mm_D1.17mm_Horizontal -> Fuse:Fuseholder_Clip-5x20mm_Littelfuse_520_Inline_P20.50x5.80mm_D1.30mm_Horizontal
Connections:
- net at C6.2, D3.1 (K), F2.1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: now also R2.2; no longer D4.2 (A)
- net at C1.2, C2.1, C3.2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: now also D4.2 (A), D5.1 (K); no longer R1.2, R2.1
- net at C5.1, D2.2 (A), F1.1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: now also R1.1; no longer D5.1 (K)
- net at D5.2 (A): now also R1.2; no longer R1.1
- net at D4.1 (K): now also R2.1; no longer R2.2
Other:
- moved on the sheet: R1, R2
